Commit message: feat: p4-1 lidarをharmonicネイティブに移行

File: mini_pupper_description/urdf/mini_pupper_2/mini_pupper_description.urdf.xacro (robot description, xacro)
@@ -1092,10 +1092,12 @@
   <gazebo reference="lidar_link">
     <material>Gazebo/FlatBlack</material>
-    <sensor type="ray" name="lidar">
+    <sensor type="gpu_lidar" name="lidar">
       <always_on>true</always_on>
       <update_rate>30</update_rate>
       <pose>0 0 0 0 0 0</pose>
       <visualize>false</visualize>
-      <ray>
+      <topic>scan</topic>
+      <gz_frame_id>lidar_link</gz_frame_id>
+      <lidar>
         <scan>
           <horizontal>
@@ -1116,6 +1118,6 @@
           <stddev>0.004</stddev>
         </noise>
-      </ray>
-      <plugin name="gazebo_ros_lidar_controller" filename="libgazebo_ros_ray_sensor.so">
+      </lidar>
+      <!-- <plugin name="gazebo_ros_lidar_controller" filename="libgazebo_ros_ray_sensor.so">
         <ros>
           <remapping>~/out:=/scan</remapping>
@@ -1123,5 +1125,5 @@
         <output_type>sensor_msgs/LaserScan</output_type>
         <frame_name>lidar_link</frame_name>
-      </plugin>
+      </plugin> -->
     </sensor>
   </gazebo>
@@ -1161,5 +1163,5 @@
   </gazebo>
   <!-- Simulated camera mounted to the front body -->
-  <link name="camera_link">
+  <!-- <link name="camera_link">
     <visual>
       <geometry>
@@ -1170,11 +1172,11 @@
       </material>
     </visual>
-  </link>
-  <joint name="bodyfront_camera_joint" type="fixed">
+  </link> -->
+  <!-- <joint name="bodyfront_camera_joint" type="fixed">
     <parent link="Body_front"/>
     <child link="camera_link"/>
     <origin xyz="0.02 0 0.02" rpy="0 0 0"/>
-  </joint>
-  <gazebo reference="camera_link">
+  </joint> -->
+  <!-- <gazebo reference="camera_link">
     <sensor type="camera" name="sim_camera">
       <always_on>true</always_on>
@@ -1193,5 +1195,4 @@
         </clip>
       </camera>
-      <!-- Gazebo ROS plugin to publish /image_raw -->
       <plugin name="camera_controller" filename="libgazebo_ros_camera.so">
         <always_on>true</always_on>
@@ -1199,8 +1200,7 @@
         <frame_name>camera_link</frame_name>
         <image_topic_name>/image_raw</image_topic_name>
-        <!-- camera_info omitted to disable /camera_info -->
       </plugin>
     </sensor>
-  </gazebo>
+  </gazebo> -->
   <xacro:mini_pupper_ros2_control use_gazebo_hardware="$(arg use_gazebo_hardware)" />
   <!-- Conditional debug support stand -->
